File: PCB/PCB.kicad_pcb (KiCad board)
At the start: 4 copper layers, 80 x 100 mm, 74 parts, among them Q1 Si1308EDL, U1 DS3231MZ+, U11 FS8205A_C2830320, U12 DW01A_C351410, U13 BC817-40,215, U14 FPC-05F-24PH20, U15 ESP32-C3FH4, U16 MC-403L68-Z10, U2 ATGM336H-7N76, U21 TS1103S-12X12X6_0SMD, U22 TS1103S-12X12X6_0SMD, U23 TS1103S-12X12X6_0SMD, U24 TS1103S-12X12X6_0SMD, U25 TS1103S-12X12X6_0SMD, U3 QMC5883P, U4 LCM1027A2445F, U5 BWGNSCNX25-25W4, U6 BS-02-A1AJ006, U7 MAX17048G+T10, U8 ME6211C33M5G-N, U9 TP4056-42-ESOP8, X1 Q22FA12800101

Commit message: upd
Parts:
- BT1: footprint Connector_JST:JST_EH_B2B-EH-A_1x02_P2.50mm_Vertical -> footprint:CONN-TH_S2B-XH-A-LF-SN
- moved BT1 34.8 mm to (100.0, 125.6), turned to -90 degrees
- moved U21 0.33 mm to (65.4, 104.3)
Routing:
- net VBAT+: track 39.3 -> 64.2 mm
- net Net-(BT1--): track 34.5 -> 53.1 mm
- net /SQW_RTC: track 61.3 -> 62.4 mm
